File: AxxSolder_hardware/AxxSolder.kicad_pcb (KiCad board)
At the start: 2 copper layers, 40 x 78.3 mm, 134 parts, among them IC2 OPA2387DSGT, IC3 LMR54406DBVR, IC5 TPD4E1U06DBVR, IC6 STUSB4500QTR, IC8 LTC4440AHMS8E, J1 284391-7, J2 Conn_01x02, J3 USB4105-GF-A, J4 61300611821, Q1 STL9P3LLH6, Q3 2N7002NXAKR, U1 LD1117S33TR_SOT223, U2 PEC11L-4220F-S0015, U3 BSC014N04LS, U5 RP2040, U6 W25Q128JVS, Y1 ABM8-272-T3

Commit message: Cleanup
Parts:
- added D12: LED, LED_SMD:LED_0603_1608Metric, B.Cu at (69.7, 94.5)
- added D13: LED, LED_SMD:LED_0603_1608Metric, F.Cu at (65.6, 66.4)
- added D14: LED, LED_SMD:LED_0603_1608Metric, B.Cu at (75.6, 97.7)
- added D15: LED, LED_SMD:LED_0603_1608Metric, B.Cu at (77.8, 97.2)
- added D16: LED, LED_SMD:LED_0603_1608Metric, B.Cu at (86.0, 71.2)
- added R47: 4k7, Resistor_SMD:R_0603_1608Metric, B.Cu at (69.6, 95.9)
- added R48: 4k7, Resistor_SMD:R_0603_1608Metric, F.Cu at (64.8, 64.2)
- added R49: 4k7, Resistor_SMD:R_0603_1608Metric, B.Cu at (77.8, 95.8)
- added R50: 4k7, Resistor_SMD:R_0603_1608Metric, B.Cu at (74.1, 96.4)
- added R51: 4k7, Resistor_SMD:R_0603_1608Metric, B.Cu at (84.4, 69.8)
- moved TP16 29.1 mm to (91.5, 99.7), turned to -90 degrees
- moved TP15 28.2 mm to (90.2, 97.5), turned to -90 degrees
- moved C2 8.72 mm to (72.5, 79.7), turned to 0 degrees
- moved C8 8.13 mm to (68.3, 88.4), turned to 90 degrees
- moved U1 5.72 mm to (70.2, 84.9)
- moved C7 5.40 mm to (69.8, 88.4)
- moved C1 3.29 mm to (68.2, 79.7), turned to 180 degrees
- moved FID1 2.65 mm to (65.5, 69.5)
- moved FID6 2.65 mm to (65.5, 69.5)
- moved C18 2.56 mm to (83.2, 100.1), turned to 180 degrees
- moved D7 2.54 mm to (69.7, 91.8)
- moved R28 2.43 mm to (73.2, 90.9)
- moved R33 2.42 mm to (73.2, 92.4)
- moved C19 1.31 mm to (86.3, 98.5), turned to 0 degrees
- moved L1 1.22 mm to (74.3, 85.3), turned to -90 degrees
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Connections:
- U5 pad 30: /Handle_inp1 -> /LED1
- U5 pad 31: /Handle_inp2 -> /LED2
- U5 pad 32: /Stand_inp -> unconnected-(U5-GPIO21-Pad32)
- U5 pad 35: unconnected-(U5-GPIO23-Pad35) -> /Handle_inp1
- U5 pad 36: unconnected-(U5-GPIO24-Pad36) -> /Handle_inp2
- U5 pad 37: /Heater -> /Stand_inp
- U5 pad 38: /TC -> /Heater
- U5 pad 39: /CURRENT -> /TC
- U5 pad 40: /VBUS_IN -> /CURRENT
- U5 pad 41: unconnected-(U5-GPIO29_ADC3-Pad41) -> /VBUS_IN
Routing:
- net (no net): track 52.0 -> 0.00 mm
- net GND: track 254.7 -> 205.4 mm, vias 79 -> 96
- net /BLUE: track 10.9 -> 2.84 mm
- net +3.3V: track 204.8 -> 196.8 mm
- net /SWDIO: track 48.9 -> 45.8 mm, vias 3 -> 1
- net /LED2: track 0.00 -> 2.98 mm
- net /SWCLK: track 54.2 -> 51.3 mm
- net /LED1: track 0.00 -> 2.77 mm
- net /VBUS_IN: track 27.4 -> 24.8 mm
- net /VCCA: track 6.71 -> 4.17 mm
- net /Stand_inp: track 25.3 -> 23.2 mm
- net /Handle_inp2: track 24.8 -> 22.7 mm
- net /Handle_inp1: track 28.8 -> 26.7 mm
- net Net-(D14-K): track 0.00 -> 1.65 mm
- net /VBUS: track 22.5 -> 24.0 mm
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- removed copper zone on B.Cu, net +7.5V

Commit message: Cleanup
Parts:
- C32, C33, R38: moved to F.Cu
- moved R48 5.74 mm to (67.2, 69.3), turned to 0 degrees
- moved R38 2.73 mm to (80.1, 81.3), turned to 180 degrees
- moved C32 2.26 mm to (83.4, 80.5), turned to -90 degrees
- moved C33 2.26 mm to (84.9, 80.5), turned to -90 degrees
- moved FID1 1.25 mm to (64.8, 70.5)
- moved FID6 1.25 mm to (64.8, 70.5)
- moved D13 1.08 mm to (66.4, 67.1), turned to 90 degrees
- moved C30 0.27 mm to (83.5, 86.8)
Routing:
- net GND: track 205.4 -> 92.4 mm, vias 96 -> 90
- net +3.3V: track 196.8 -> 141.2 mm, vias 18 -> 16
- net /SDA: track 54.5 -> 64.1 mm
- net /SCL: track 54.3 -> 63.8 mm
- net Net-(IC8-TG): track 13.6 -> 7.63 mm
- net /BLUE: track 2.84 -> 0.00 mm
- net /RED: track 15.4 -> 12.8 mm
- net +7.5V: track 117.4 -> 115.9 mm, vias 3 -> 4
- net /SW2: track 26.2 -> 27.8 mm
- net /USB_D+: track 44.4 -> 45.6 mm
- net /Handle_inp1: track 26.7 -> 26.0 mm
- net /Heater: track 28.3 -> 27.8 mm, vias 0 -> 1
- net /ENC_A: track 34.6 -> 34.0 mm
- net /USB_D-: track 43.4 -> 44.0 mm
- net /Handle_inp2: track 22.7 -> 22.2 mm
