File: AxxSolder_hardware/AxxSolder.kicad_pcb (KiCad board)
At the start: 2 copper layers, 40 x 78.3 mm, 144 parts, among them IC2 OPA2387DSGT, IC3 LMR54406DBVR, IC5 TPD4E1U06DBVR, IC6 STUSB4500QTR, IC8 LTC4440AHMS8E, J1 284391-7, J2 Conn_01x02, J3 USB4105-GF-A, J4 61300611821, Q1 STL9P3LLH6, Q3 2N7002NXAKR, U1 LD1117S33TR_SOT223, U2 PEC11L-4220F-S0015, U3 BSC014N04LS, U5 RP2040, U6 W25Q128JVS, Y1 ABM8-272-T3

Commit message: Best work yet
Parts:
- removed C10: 10u, Capacitor_SMD:C_0603_1608Metric
- removed J2: Conn_01x02, Connector_PinHeader_2.54mm:PinHeader_1x02_P2.54mm_Vertical
- added R52: 4k7, Resistor_SMD:R_0603_1608Metric, F.Cu at (144.2, 148.2)
- added TP1: USR1, TestPoint:TestPoint_Pad_D1.0mm, B.Cu at (141.6, 149.9)
- C1, C14, C2, C25, C26, C27, C39, C4, C44, C6, D5, D6, D8, FID1, IC2, R10, R18, R19, R2, R20, R22, R25, R29, R3, R6, R9, TP7, TP8, U1: moved to B.Cu
- C11, C12, C13, C3, C32, C33, C34, C35, C5, C7, C8, D10, D14, D15, D16, D9, FID5, FID6, IC3, IC6, IC8, L1, LS1, R11, R14, R26, R27, R45, R46, R49, R50, R51, R7, R8, U3: moved to F.Cu
- D4: value SMF4L24AT1G -> LED; footprint footprints:SODFL3619X98N -> LED_SMD:LED_0603_1608Metric; moved to F.Cu
- J1: value 284391-7 -> 691243310007; footprint custom_connectors:CONN7_284391-7_TEC -> custom_connectors:691243310007
- J4: value 61300611821 -> Conn_01x07_Pin; footprint Connector_PinHeader_2.54mm:PinHeader_1x06_P2.54mm_Vertical -> Connector_PinHeader_2.54mm:PinHeader_1x07_P2.54mm_Vertical; moved to F.Cu
- U6: value W25Q128JVS -> W25Q16JVSSIQ
- moved FID1 127.1 mm to (146.7, 167.3), turned to 180 degrees
- moved FID6 127.1 mm to (146.7, 167.3), turned to 0 degrees
- moved FID5 97.4 mm to (176.1, 81.9), turned to 0 degrees
- moved J4 93.8 mm to (148.2, 139.3)
- moved D4 89.9 mm to (141.2, 148.2), turned to 180 degrees
- moved R48 89.3 mm to (133.1, 121.7), turned to 180 degrees
- moved D13 86.4 mm to (133.8, 119.5), turned to 90 degrees
- moved R50 85.4 mm to (144.2, 145.2), turned to 0 degrees
- moved R49 83.7 mm to (144.2, 146.7), turned to 0 degrees
- moved D3 82.0 mm to (134.5, 109.3), turned to 180 degrees
- moved D14 81.0 mm to (141.3, 145.2), turned to 180 degrees
- moved Y1 80.8 mm to (135.1, 149.4), turned to 180 degrees
- moved D15 80.4 mm to (141.2, 146.7)
- moved C36 78.1 mm to (136.8, 146.9), turned to 0 degrees
- moved J3 76.9 mm to (138.8, 102.6)
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Connections:
- D4 pad 1: VDD -> Net-(D4-K)
- D4 pad 2: GND -> /LED3
- IC5 pad 1: /CC1 -> /USB_D-
- IC5 pad 4: /USB_D- -> /CC2
- IC5 pad 6: /CC2 -> /CC1
- J1 pad 5: /BLUE -> GND
- J1 pad 6: GND -> /BLUE
- J4 pad 1: /SWCLK -> /~{USB_BOOT}
- J4 pad 2: /SWDIO -> GND
- J4 pad 3: GND -> /SWCLK
- J4 pad 4: +3.3V -> /SWDIO
- U2 pad 1: /SW1 -> +3.3V
- U2 pad 2: +3.3V -> /SW1
- U5 pad 12: /SW1 -> unconnected-(U5-GPIO9-Pad12)
- U5 pad 13: /ENC_A -> /SCL
- U5 pad 14: /SPI_RST -> /SDA
- U5 pad 15: /SPI_DC -> /LED1
- U5 pad 16: /SPI_CS -> /LED2
- U5 pad 17: /SPI_SCK -> /LED3
- U5 pad 18: /SPI_MOSI -> /USR1
- U5 pad 2: /SDA -> /SPI_RST
- U5 pad 27: unconnected-(U5-GPIO16-Pad27) -> /SW3
- U5 pad 28: /USART_RX -> /SW2
- U5 pad 29: /USART_TX -> /ENC_B
- U5 pad 3: /SCL -> /SPI_DC
- U5 pad 30: /LED1 -> /ENC_A
- U5 pad 31: /LED2 -> /SW1
- U5 pad 32: unconnected-(U5-GPIO21-Pad32) -> /Handle_inp1
- U5 pad 34: unconnected-(U5-GPIO22-Pad34) -> /Handle_inp2
- U5 pad 35: /Handle_inp1 -> /Stand_inp
- U5 pad 36: /Handle_inp2 -> /Buzzer
- U5 pad 37: /Stand_inp -> /Heater
- U5 pad 38: /Heater -> /CURRENT
- U5 pad 4: /Buzzer -> /SPI_CS
- U5 pad 40: /CURRENT -> /VBUS_IN
- U5 pad 41: /VBUS_IN -> unconnected-(U5-GPIO29_ADC3-Pad41)
- U5 pad 5: /SW3 -> /SPI_SCK
- U5 pad 6: /SW2 -> /SPI_MOSI
- U5 pad 7: unconnected-(U5-GPIO5-Pad7) -> /USART_RX
- U5 pad 8: /ENC_B -> /USART_TX
Routing:
- net GND: track 205.4 -> 34.7 mm, vias 96 -> 81
- net +7.5V: track 117.4 -> 34.4 mm, vias 3 -> 1
- net +3.3V: track 196.8 -> 274.6 mm
- net /SWDIO: track 45.8 -> 80.2 mm, vias 1 -> 2
- net /RED: track 15.4 -> 49.0 mm, vias 0 -> 1
- net Net-(IC2B--): track 17.5 -> 43.6 mm, vias 0 -> 2
- net Net-(IC2B-+): track 15.1 -> 40.5 mm, vias 1 -> 2
- net /SWCLK: track 51.3 -> 71.7 mm, vias 1 -> 2
- net /Buzzer: track 29.7 -> 10.6 mm, vias 2 -> 0
- net /GREEN: track 9.85 -> 28.9 mm
- net Net-(IC2A--): track 31.7 -> 12.8 mm, vias 2 -> 1
- net /H_sense1: track 11.5 -> 29.2 mm
- net /SCL: track 54.3 -> 36.6 mm
- net Net-(Q1-G): track 5.27 -> 22.9 mm
- net /USB_D+: track 44.4 -> 28.0 mm, vias 3 -> 2
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- added copper zone on F.Cu, net +7.5V
- added copper zone on F.Cu, net /RED
- added copper zone on F.Cu, net Net-(IC3-SW)
- added copper zone on F.Cu, net VDD
- removed copper zone on B.Cu, net +1V1
- removed copper zone on B.Cu, net +3.3V
- removed copper zone on F.Cu, net +3.3V
- removed copper zone on B.Cu, net /RED
- removed copper zone on B.Cu, net /VDD_IN
- removed copper zone on B.Cu, net Net-(IC3-SW)
Other:
- board size 40 x 78.3 mm -> 50 x 70 mm

Commit message: Perfection
Parts:
- removed U1: LD1117S33TR_SOT223, Package_TO_SOT_SMD:SOT-223-3_TabPin2
- added C10: 100p, Capacitor_SMD:C_0603_1608Metric, B.Cu at (115.9, 125.7)
- added U4: AP2210K-3.3, Package_TO_SOT_SMD:SOT-23-5, B.Cu at (116.1, 128.5)
- J4: moved to B.Cu
- moved FID5 89.9 mm to (133.2, 160.9), turned to 90 degrees
- moved R38 5.75 mm to (118.2, 123.6)
- moved C1 3.68 mm to (116.3, 131.3), turned to 180 degrees
- moved C2 3.66 mm to (118.5, 128.1), turned to -90 degrees
- moved R6 0.50 mm to (112.0, 119.3)
- moved R23 0.50 mm to (117.1, 133.6), turned to -90 degrees
- moved Q3 0.30 mm to (116.7, 136.9)
- moved D4 0.25 mm to (141.2, 148.5)
- moved R34 0.25 mm to (120.0, 136.6)
- moved R37 0.25 mm to (120.0, 138.1)
- moved R52 0.25 mm to (144.2, 148.4)
- moved D15 0.15 mm to (141.2, 146.8)
- moved R49 0.15 mm to (144.2, 146.8)
- turned J4 to 180 degrees
Routing:
- net +3.3V: track 274.6 -> 251.8 mm, vias 18 -> 17
- net +1V1: track 17.4 -> 9.08 mm
- net GND: track 34.7 -> 41.5 mm, vias 81 -> 88
- net /Heater: track 38.3 -> 35.7 mm
- net Net-(U4-BYP): track 0.00 -> 1.67 mm
- net +7.5V: track 34.4 -> 36.0 mm
- net /SWCLK: track 71.7 -> 70.9 mm
- net /GREEN: track 28.9 -> 29.5 mm
- net Net-(R21-Pad1): track 8.69 -> 9.31 mm
- net Net-(IC2B-+): track 40.5 -> 39.9 mm
- added copper zone on B.Cu, net +1V1
Other:
- board text added: "3V3"
- board text added: "B"
- board text added: "G"
- board text added: "GND"
- board text added: "H1"
- board text added: "H2"
- board text added: "R"
- board text added: "RX"
- board text added: "S1"
- board text added: "SWCLK"
- board text added: "SWDIO"
- board text added: "TX"
