File: AxxSolder_hardware/AxxSolder.kicad_pcb (KiCad board)
At the start: 2 copper layers, 50 x 70 mm, 145 parts, among them IC2 OPA2387DSGT, IC3 LMR54406DBVR, IC5 TPD4E1U06DBVR, IC6 STUSB4500QTR, IC8 LTC4440AHMS8E, J1 691243310007, J3 USB4105-GF-A, J4 Conn_01x07_Pin, Q1 STL9P3LLH6, Q3 2N7002NXAKR, U2 PEC11L-4220F-S0015, U3 BSC014N04LS, U4 AP2210K-3.3, U5 RP2040, U6 W25Q16JVSSIQ, Y1 ABM8-272-T3

Commit message: Ordered this one
Parts:
- added C15: 100n, Capacitor_SMD:C_0603_1608Metric, B.Cu at (140.7, 101.8)
- added Q2: 2N7002NXAKR, footprints:SOT95P230X110-3N, F.Cu at (141.8, 150.8)
- added Q4: 2N7002NXAKR, footprints:SOT95P230X110-3N, F.Cu at (141.8, 147.3)
- added Q5: 2N7002NXAKR, footprints:SOT95P230X110-3N, B.Cu at (140.6, 144.9)
- added R53: 1M, Resistor_SMD:R_0603_1608Metric, B.Cu at (140.7, 103.3)
- C30, R42: moved to F.Cu
- D12, D13, D14, D16, D4: value LED -> 150060VS75000
- D15: value LED -> 150060VS75000; moved to B.Cu
- D5, D6, D7, D8: value BAT54S -> BAT54SLT1G
- R47, R50, R52: value 4k7 -> 100
- R48, R51: value 4k7 -> 1k5; footprint Resistor_SMD:R_0603_1608Metric -> Resistor_SMD:R_0603_1608Metric_Pad0.98x0.95mm_HandSolder
- R49: value 4k7 -> 100; moved to B.Cu
- U4: value AP2210K-3.3 -> AP2210K-3.3TRG1
- moved C37 9.33 mm to (115.7, 106.8), turned to 90 degrees
- moved R42 8.81 mm to (102.5, 113.0), turned to 90 degrees
- moved C35 8.44 mm to (120.2, 103.5), turned to 90 degrees
- moved D14 7.69 mm to (146.2, 151.1), turned to -90 degrees
- moved C34 7.27 mm to (121.8, 103.5), turned to 90 degrees
- moved D15 6.95 mm to (140.1, 139.9), turned to 90 degrees
- moved R6 6.80 mm to (110.0, 112.8)
- moved R49 5.91 mm to (141.6, 141.6), turned to -90 degrees
- moved D4 4.20 mm to (144.5, 151.1), turned to -90 degrees
- moved F1 3.99 mm to (126.8, 106.0)
- moved C30 3.94 mm to (118.2, 111.1), turned to -90 degrees
- moved R50 3.52 mm to (146.2, 148.1), turned to 90 degrees
- moved R4 3.50 mm to (110.0, 115.8)
- moved D10 3.27 mm to (102.7, 106.2), turned to 90 degrees
- moved FID2 0.70 mm to (102.5, 101.8)
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Connections:
- C11 pad 1: /VBUS -> GND
- C11 pad 2: GND -> /VBUS
- C12 pad 1: Net-(IC6-VREG_2V7) -> GND
- C12 pad 2: GND -> Net-(IC6-VREG_2V7)
- C13 pad 1: Net-(IC6-VREG_1V2) -> GND
- C13 pad 2: GND -> Net-(IC6-VREG_1V2)
- C30 pad 1: /RED -> /BOOST
- C30 pad 2: /BOOST -> /RED
- C34 pad 1: GND -> VDD
- C34 pad 2: VDD -> GND
- C35 pad 1: GND -> VDD
- C35 pad 2: VDD -> GND
- C5 pad 1: GND -> VDD
- C5 pad 2: VDD -> GND
- C7 pad 1: GND -> +7.5V
- C7 pad 2: +7.5V -> GND
- C8 pad 1: GND -> +7.5V
- C8 pad 2: +7.5V -> GND
- C9 pad 1: Net-(C9-Pad1) -> /VDD_IN
- C9 pad 2: /VDD_IN -> Net-(C9-Pad2)
- D14 pad 2: /LED1 -> +3.3V
- D15 pad 2: /LED2 -> +3.3V
- D4 pad 2: /LED3 -> +3.3V
- J1 pad 5: GND -> /BLUE
- J1 pad 6: /BLUE -> GND
- J3 pad SH1: GND -> Net-(J3-SHELL_GND)
- J3 pad SH2: GND -> Net-(J3-SHELL_GND)
- J3 pad SH3: GND -> Net-(J3-SHELL_GND)
- J3 pad SH4: GND -> Net-(J3-SHELL_GND)
- R13 pad 2: Net-(C9-Pad1) -> Net-(C9-Pad2)
- R49 pad 2: GND -> Net-(Q5-D)
- R50 pad 2: GND -> Net-(Q4-D)
- R52 pad 2: GND -> Net-(Q2-D)
Routing:
- net Net-(J3-SHELL_GND): track 0.00 -> 20.2 mm
- net GND: track 41.5 -> 26.0 mm, vias 88 -> 79
- net /VBUS: track 25.5 -> 38.2 mm, vias 2 -> 9
- net +3.3V: track 251.8 -> 260.7 mm
- net Net-(IC2B--): track 43.6 -> 50.6 mm
- net +7.5V: track 36.0 -> 30.2 mm
- net /BLUE: track 9.06 -> 13.9 mm
- net VDD: track 25.6 -> 21.1 mm
- net Net-(Q2-D): track 0.00 -> 4.22 mm
- net Net-(Q5-D): track 0.00 -> 4.09 mm
- net Net-(Q4-D): track 0.00 -> 3.91 mm
- net Net-(IC2B-+): track 39.9 -> 43.5 mm
- net /RED: track 49.0 -> 51.6 mm, vias 1 -> 0
- net Net-(C9-Pad2): track 0.00 -> 2.22 mm
- net Net-(C9-Pad1): track 2.22 -> 0.00 mm
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- added copper zone on B.Cu, net +3.3V
- added copper zone on F.Cu, net /BLUE
- added copper zone on B.Cu, net /VDD_IN
- removed copper zone on B.Cu, net /BLUE
