File: AxxSolder_hardware/AxxSolder.kicad_sch (KiCad schematic)
At the start: 143 parts, among them IC1 TLV76733DRVR, IC2 OPA2387DSGT, IC3 LMR54406DBVR, IC4 STM32G431CBT6, IC5 TPD4E1U06DBVR, IC6 STUSB4500QTR, IC7 MAX16171ATA_VY+T, IC8 LTC4440AHMS8E, IC9 INA281A5QDBVRQ1, J1 USB4110-GF-A, J2 691243110009, J3 TSW-102-07-T-S, J4 61300611821, J5 TSW-102-07-T-S, J6 TSW-102-07-T-S, Q1 STL9P3LLH6, Q2 STL10N3LLH5, Q3 2N7002NXAKR, U2 PEC11J-9215F-S0015, U3 BSC014N04LS

Commit message: Replace MCU with RP2040, new PCB layout
Parts:
- removed C14, C15, C16, C17: 100n, Capacitor_SMD:C_0603_1608Metric, symbol Device:C_Small
- removed C31: 10u, Capacitor_SMD:C_0603_1608Metric, symbol Device:C_Small
- removed F2: SF-2410FP100W-2, footprints:SF2410FP100W2, symbol SF-2410FP100W-2:SF-2410FP100W-2
- removed IC1: TLV76733DRVR, footprints:SON65P200X200X80-7N, symbol TLV76733DRVR:TLV76733DRVR
- removed IC4: STM32G431CBT6, footprints:QFP50P900X900X160-48N, symbol STM32G431CBT6:STM32G431CBT6
- removed IC7: MAX16171ATA_VY+T, footprints:SON50P300X200X80-9N, symbol MAX16171ATA_VY+T:MAX16171ATA_VY+T
- removed IC9: INA281A5QDBVRQ1, footprints:SOT95P280X145-5N, symbol INA281A5QDBVRQ1:INA281A5QDBVRQ1
- removed J2: 691243110009, footprints:691243110009, symbol 691243110009:691243110009
- removed J3: TSW-102-07-T-S, Connector_PinHeader_2.54mm:PinHeader_1x02_P2.54mm_Vertical, symbol TSW-102-07-T-S:TSW-102-07-T-S
- removed J5, J6: TSW-102-07-T-S, footprints:TSW-102-XX-YY-S, symbol TSW-102-07-T-S:TSW-102-07-T-S
- removed Q2: STL10N3LLH5, footprints:STL10N3LLH5, symbol STL10N3LLH5:STL10N3LLH5
- removed R44: 1M, Resistor_SMD:R_0805_2012Metric, symbol Device:R_Small
- removed R45: 100m, Resistor_SMD:R_0805_2012Metric, symbol Device:R_Small
- removed S1: ADTSM644RVTR, footprints:ADTSM644RVTR, symbol ADTSM644KVTR:ADTSM644KVTR
- removed TP1, TP14, TP2, TP5, TP6: DIAG_TP, TestPoint:TestPoint_Pad_D1.0mm, symbol Connector:TestPoint
- removed TP12: GND_TP, TestPoint:TestPoint_Pad_D1.0mm, symbol Connector:TestPoint
- removed TP13: DIAG_TP, Connector_PinSocket_2.54mm:PinSocket_1x01_P2.54mm_Vertical, symbol Connector:TestPoint
- removed TP3: 3.3V_TP, TestPoint:TestPoint_Pad_D1.0mm, symbol Connector:TestPoint
- removed TP9: Current_TP, TestPoint:TestPoint_Pad_D1.0mm, symbol Connector:TestPoint
- removed U1: ~, footprints:Adafruit_240x320_TFT, symbol Adafruit_240x320_TFT:Adafruit_240x320_TFT
- removed U2: PEC11J-9215F-S0015, footprints:PEC11J9215FS0015, symbol PEC11J-9215F-S0015:PEC11J-9220F-S0015
- added C36, C38: 15p, Capacitor_SMD:C_0603_1608Metric, symbol Device:C
- added C39, C40, C41, C43, C45, C46, C47, C48, C50: 100n, Capacitor_SMD:C_0603_1608Metric, symbol Device:C
- added C42, C44: 1u, Capacitor_SMD:C_0603_1608Metric, symbol Device:C
- added H3, H4, H5, H6: MountingHole, MountingHole:MountingHole_2.5mm, symbol Mechanical:MountingHole
- added J2: Conn_01x02, Connector_PinHeader_2.54mm:PinHeader_1x02_P2.54mm_Vertical, symbol Connector_Generic:Conn_01x02
- added J7: Conn_01x07_Pin, Connector_PinHeader_2.54mm:PinHeader_1x07_P2.54mm_Vertical, symbol Connector:Conn_01x07_Pin
- added R16, R43: 1k, Resistor_SMD:R_0603_1608Metric, symbol Device:R
- added R44: 10k, Resistor_SMD:R_0603_1608Metric, symbol Device:R
- added R45, R46: 27, Resistor_SMD:R_0603_1608Metric, symbol Device:R
- added SW1: PEC11L-4220F-S0015, custom:PEC11L-4xxxF-Sxxxx_BRN, symbol custom:PEC11L-4220F-S0015
- added U1: LD1117S33TR_SOT223, Package_TO_SOT_SMD:SOT-223-3_TabPin2, symbol Regulator_Linear:LD1117S33TR_SOT223
- added U5: RP2040, custom:RP2040-QFN-56, symbol MCU_RaspberryPi_RP2040:RP2040
- added U6: W25Q128JVS, Package_SO:SOIC-8_5.23x5.23mm_P1.27mm, symbol Memory_Flash:W25Q128JVS
- added U7: WS3-013992, custom:WS-13992, symbol custom:WS3-013992
- added Y1: ABM8-272-T3, Crystal:Crystal_SMD_3225-4Pin_3.2x2.5mm, symbol Device:Crystal_GND24
- C37: footprint CAPAE830X1050N -> footprints:CAPAE830X1050N
- IC3, IC5: footprint SOT95P280X145-6N -> footprints:SOT95P280X145-6N
- J1: footprint USB4110GFA -> footprints:USB4110GFA
Connections:
- net NRST is gone; now on net GND: J4.3 (Pin_3)
- net VDD_IN_USBCPD is gone; now on net VDD_IN: C9.2, Q1.5 (D), R17.2
- net +3.3V: now also J4.4 (Pin_4), R35.1, C39.1, C43.1, C44.1, C45.1, C46.1, C47.1, C48.1, C50.1, R44.1, SW1.2, U1.2 (VO), U5.1 (IOVDD), U5.10 (IOVDD), U5.22 (IOVDD), U5.33 (IOVDD), U5.42 (IOVDD), U5.44 (VREG_IN), U5.48 (USB_VDD), U5.49 (IOVDD), U6.8 (VCC), U7.1 (VCC); no longer J4.2 (Pin_2), R35.2
- net +7.5V: now also U1.3 (VI)
- net BLUE: now also J7.5 (Pin_5)
- net Buzzer: now also U5.13 (GPIO10)
- net CURRENT: now also U5.39 (GPIO27_ADC1)
- net ENC_A: now also SW1.B, U5.28 (GPIO17)
- net ENC_B: now also R35.2, SW1.A, U5.29 (GPIO18); no longer R35.1
- net GND: now also J1.S1 (SHIELD), C36.2, C38.2, C39.2, C40.2, C41.2, C42.2, C43.2, C44.2, C45.2, C46.2, C47.2, C48.2, C50.2, J2.2 (Pin_2), J7.6 (Pin_6), SW1.C, U1.1 (GND), U5.19 (TESTEN), U5.57 (GND), U6.4 (GND), U7.2 (GND), Y1.2, Y1.4; no longer J4.1 (Pin_1)
- net GREEN: now also J7.4 (Pin_4)
- net H_sense1: now also J7.3 (Pin_3)
- net H_sense2: now also J7.2 (Pin_2)
- net Handle_inp1: now also U5.30 (GPIO19)
- net Handle_inp2: now also U5.31 (GPIO20)
- net Heater: now also U5.37 (GPIO25)
- net RED: now also J7.7 (Pin_7)
- net SCL: now also U5.3 (GPIO1)
- net SDA: now also U5.2 (GPIO0)
- net SPI_CS: now also U5.15 (GPIO12), U7.6 (CS)
- net SPI_DC: now also U5.18 (GPIO15), U7.7 (DC)
- net SPI_MOSI: now also U5.14 (GPIO11), U7.4 (DIN)
- net SPI_RST: now also U5.17 (GPIO14), U7.8 (RST)
- net SPI_SCK: now also U5.16 (GPIO13), U7.5 (CLK)
- net SW1: now also SW1.1, U5.9 (GPIO7)
- net SW2: now also U5.11 (GPIO8)
- net SW3: now also U5.12 (GPIO9)
- net SWCLK: now also J4.1 (Pin_1), U5.24 (SWCLK); no longer J4.4 (Pin_4)
- net SWDIO: now also J4.2 (Pin_2), U5.25 (SWD); no longer J4.5 (Pin_5)
- net S_sense: now also J7.1 (Pin_1)
- net Stand_inp: now also U5.32 (GPIO21)
- net TC: now also U5.38 (GPIO26_ADC0)
- net USART_RX: now also J4.5 (Pin_5), U5.5 (GPIO3)
- net USART_TX: now also U5.4 (GPIO2)
- net USB_D+: now also R45.1
- net USB_D-: now also R46.1
- net USR1: now also U5.6 (GPIO4)
- net VBUS_IN: now also U5.40 (GPIO28_ADC2)
- net VCCA: now also U5.43 (ADC_AVDD)
- net VDD: now also F1.2; no longer F1.1
- net VDD_IN: now also F1.1; no longer F1.2
- new net: C38.1, R16.2, Y1.3
- new net: R45.2, U5.47 (USB_DP)
- new net: R46.2, U5.46 (USB_DM)
- new net +1V1: C40.1, C41.1, C42.1, U5.23 (DVDD), U5.45 (VREG_VOUT), U5.50 (DVDD)
- new net NC: U7.3 (NC)
- new net QSPI_SCLK: U5.52 (QSPI_SCLK), U6.6 (CLK)
- new net QSPI_SD0: U5.53 (QSPI_SD0), U6.5 (DI(IO0))
- new net QSPI_SD1: U5.55 (QSPI_SD1), U6.2 (DO(IO1))
- new net QSPI_SD2: U5.54 (QSPI_SD2), U6.3 (IO2)
- new net QSPI_SD3: U5.51 (QSPI_SD3), U6.7 (IO3)
- new net QSPI_SS: R43.1, R44.2, U5.56 (QSPI_SS), U6.1 (~{CS})
- new net RUN: U5.26 (RUN)
- new net XIN: C36.1, U5.20 (XIN), Y1.1
- new net XOUT: R16.1, U5.21 (XOUT)
- new net ~{USB_BOOT}: J2.1 (Pin_1), R43.2
Other:
- note added: "AxxSolder V3.1 JBC Soldering Iron Controller"
- note added: "Crystal"
- note added: "DISPLAY"
- note added: "Flash"
- note added: "HGIH-SIDE DRIVER AND MOSFET"
- note added: "Make sure C10 is close to pin 44 of RP2040"
- note added: "Make sure R3 and R4 are close to RP2040"
- note added: "SCREW TERMINAL"
- note removed: "1A"
- note removed: "240x320 TFT DISPLAY"
- note removed: "AxxSolder V3.0 JBC Soldering Iron Controller"
- note removed: "EARTH"
- note removed: "HGIH-SIDE DRIVER ADN MOSFET"
- note removed: "LCD"
- note removed: "SCREW TERMINAL AND EARTH LEAK SENSE"
- note removed: "SUPPORT"
- note removed: "alt. part: RIC11-31S15D7-GSMT"
- moved on the sheet: C1, C10, C11, C12, C13, C18, C19, C2, C22, C28, C29, C30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

Commit message: Cleanup
Parts:
- removed H1, H2: MountingHole, MountingHole:MountingHole_2.5mm, symbol Mechanical:MountingHole
Changed lines of the file:
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@@
 	)
 	(symbol
-		(lib_id "Mechanical:MountingHole")
-		(at 119.38 194.945 0)
-		(unit 1)
-		(exclude_from_sim no)
-		(in_bom no)
-		(on_board yes)
-		(dnp no)
-		(property "Reference" "H1"
-			(at 118.11 191.77 0)
-			(effects
-				(font
-					(size 1.27 1.27)
-				)
-				(justify left)
-			)
-		)
-		(property "Value" "MountingHole"
-			(at 121.92 196.2149 0)
-			(effects
-				(font
-					(size 1.27 1.27)
-				)
-				(justify left)
-				(hide yes)
-			)
-		)
-		(property "Footprint" "MountingHole:MountingHole_2.5mm"
-			(at 119.38 194.945 0)
-			(effects
-				(font
-					(size 1.27 1.27)
-				)
-				(hide yes)
-			)
-		)
-		(property "Datasheet" "~"
-			(at 119.38 194.945 0)
-			(effects
-				(font
-					(size 1.27 1.27)
-				)
-				(hide yes)
-			)
-		)
-		(property "Description" ""
-			(at 119.38 194.945 0)
-			(effects
-				(font
-					(size 1.27 1.27)
-				)
-				(hide yes)
-			)
-		)
-		(property "Assembly Comment" "N/A"
-			(at 119.38 194.945 0)
-			(effects
-				(font
-					(size 1.27 1.27)
-				)
-				(hide yes)
-			)
-		)
-		(property "Manufacturing comment" "Do Not Place"
-			(at 119.38 194.945 0)
-			(effects
-				(font
-					(size 1.27 1.27)
-				)
-				(hide yes)
-			)
-		)
-		(instances
-			(project "AxxSolder"
-				(path "/d71363c3-4d90-469c-a600-831e2a7cdaef"
-					(reference "H1")
-					(unit 1)
-				)
-			)
-		)
-	)
-	(symbol
 		(lib_id "power:GND")
 		(at 166.37 86.36 0)
@@
 					(unit 1)
 				)
-			)
-		)
-	)
-	(symbol
-		(lib_id "Mechanical:MountingHole")
-		(at 124.46 194.945 0)
-		(unit 1)
-		(exclude_from_sim no)
-		(in_bom no)
-		(on_board yes)
-		(dnp no)
-		(property "Reference" "H2"
-			(at 123.19 191.77 0)
-			(effects
-				(font
-					(size 1.27 1.27)
-				)
-				(justify left)
-			)
-		)
-		(property "Value" "MountingHole"
-			(at 127 196.2149 0)
-			(effects
-				(font
-					(size 1.27 1.27)
-				)
-				(justify left)
-				(hide yes)
-			)
-		)
-		(property "Footprint" "MountingHole:MountingHole_2.5mm"
-			(at 124.46 194.945 0)
-			(effects
-				(font
-					(size 1.27 1.27)
-				)
-				(hide yes)
-			)
-		)
-		(property "Datasheet" "~"
-			(at 124.46 194.945 0)
-			(effects
-				(font
-					(size 1.27 1.27)
-				)
-				(hide yes)
-			)
-		)
-		(property "Description" ""
-			(at 124.46 194.945 0)
-			(effects
-				(font
-					(size 1.27 1.27)
-				)
-				(hide yes)
-			)
-		)
-		(property "Assembly Comment" "N/A"
-			(at 124.46 194.945 0)
-			(effects
-				(font
-					(size 1.27 1.27)
-				)
-				(hide yes)
-			)
-		)
-		(property "Manufacturing comment" "Do Not Place"
-			(at 124.46 194.945 0)
-			(effects
-				(font
-					(size 1.27 1.27)
-				)
-				(hide yes)
-			)
-		)
-		(instances
-			(project "AxxSolder"
-				(path "/d71363c3-4d90-469c-a600-831e2a7cdaef"
-					(reference "H2")
-					(unit 1)
-				)

Commit message: Cleanup
Parts:
- removed C20: 10u, Capacitor_SMD:C_0603_1608Metric, symbol Device:C_Small
- removed H3, H4, H5, H6: MountingHole, MountingHole:MountingHole_2.5mm, symbol Mechanical:MountingHole
- removed J1: USB4110-GF-A, footprints:USB4110GFA, symbol USB4110-GF-A:USB4110-GF-A
- removed J7: Conn_01x07_Pin, Connector_PinHeader_2.54mm:PinHeader_1x07_P2.54mm_Vertical, symbol Connector:Conn_01x07_Pin
- removed SW1: PEC11L-4220F-S0015, custom:PEC11L-4xxxF-Sxxxx_BRN, symbol custom:PEC11L-4220F-S0015
- removed TP4: DIAG_TP, TestPoint:TestPoint_Pad_D1.0mm, symbol Connector:TestPoint
- removed U7: WS3-013992, custom:WS-13992, symbol custom:WS3-013992
- added C14: 100n, Capacitor_SMD:C_0603_1608Metric, symbol Device:C
- added D11: 1_5inch-rgb-oled-module_asm-1110, custom_hmi:1_5inch-rgb-oled-module_asm-1110, symbol custom_interface:1_5inch-rgb-oled-module_asm-1110
- added FID4: OSHW symbol, Symbol:OSHW-Logo_5.7x6mm_Copper, symbol Mechanical:Fiducial
- added FID5: Kicad symbol, Symbol:KiCad-Logo_6mm_SilkScreen, symbol Mechanical:Fiducial
- added J1: 284391-7, custom_connectors:CONN7_284391-7_TEC, symbol custom_connectors:284391-7
- added J3: USB4105-GF-A, custom_connectors:GCT_USB4105-GF-A, symbol custom_connectors:USB4105-GF-A
- added U2: PEC11L-4220F-S0015, custom_hmi:PEC11L4220FS0015, symbol custom_interface:PEC11L-4220F-S0015
- J4: footprint footprints:RHDR6W97P0X254_1X6_1574X250X865P -> Connector_PinHeader_2.54mm:PinHeader_1x06_P2.54mm_Vertical
- TP10: value Current_TP -> Current
- TP11: value TC_TP -> TC
- TP15: value DIAG_TP -> SCL
- TP16: value DIAG_TP -> SDA
- TP17: value SW_TP -> PWM
- TP7: value DIAG_TP -> CC1
- TP8: value DIAG_TP -> CC2
Connections:
- net USR1 is gone; now on net SW2: U5.6 (GPIO4)
- net +3.3V: now also C14.1, D11.1 (VCC), U2.2 (S2)
- net BLUE: now also J1.5
- net Buzzer: now also U5.4 (GPIO2); no longer U5.13 (GPIO10)
- net CC1: now also J3.A5 (CC1)
- net CC2: now also J3.B5 (CC2)
- net ENC_A: now also C28.1, R35.2, U5.13 (GPIO10), U2.3 (A); no longer C29.1, R36.2, U5.28 (GPIO17)
- net ENC_B: now also C29.1, R36.2, U5.8 (GPIO6), U2.5 (B); no longer C28.1, R35.2, U5.29 (GPIO18)
- net GND: now also C14.2, D11.2 (GND), J1.6, J3.A1_B12 (GND), J3.B1_A12 (GND__1), J3.SH1 (SHELL_GND), J3.SH2 (SHELL_GND__1), J3.SH3 (SHELL_GND__2), J3.SH4 (SHELL_GND__3), U2.4 (C)
- net GREEN: now also J1.4
- net H_sense1: now also J1.3
- net H_sense2: now also J1.2
- net RED: now also J1.7
- net SPI_CS: now also U5.16 (GPIO13), D11.6 (CS); no longer U5.15 (GPIO12)
- net SPI_DC: now also U5.15 (GPIO12), D11.7 (DC); no longer U5.18 (GPIO15)
- net SPI_MOSI: now also U5.18 (GPIO15), D11.4 (DIN); no longer U5.14 (GPIO11)
- net SPI_RST: now also U5.14 (GPIO11), D11.8 (RST); no longer U5.17 (GPIO14)
- net SPI_SCK: now also U5.17 (GPIO14), D11.5 (CLK); no longer U5.16 (GPIO13)
- net SW1: now also U5.12 (GPIO9), U2.1 (S1); no longer U5.9 (GPIO7)
- net SW2: no longer U5.11 (GPIO8)
- net SW3: now also U5.5 (GPIO3); no longer U5.12 (GPIO9)
- net SWCLK: now also J3.B8 (SBU2)
- net SWDIO: now also J3.A8 (SBU1)
- net S_sense: now also J1.1
- net USART_RX: now also U5.28 (GPIO17); no longer U5.5 (GPIO3)
- net USART_TX: now also U5.29 (GPIO18); no longer U5.4 (GPIO2)
- net USB_D+: now also IC5.3 (IO2), J3.A6 (DP1), J3.B6 (DP2); no longer IC5.4 (IO3)
- net USB_D-: now also IC5.4 (IO3), J3.A7 (DN1), J3.B7 (DN2); no longer IC5.3 (IO2)
- net VBUS: now also J3.A4_B9 (VBUS), J3.B4_A9 (VBUS__1)
Other:
- note removed: "Version: 0x000"
- moved on the sheet: IC2C

Commit message: Cleanup
Parts:
- added FID6: Fiducial, Fiducial:Fiducial_0.75mm_Mask1.5mm, symbol Mechanical:Fiducial
Changed lines of the file:
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@@
 				(thickness 0.254)
 				(bold yes)
+				(color 0 0 255 1)
 			)
 			(justify left bottom)
@@
 			(font
 				(size 1.27 1.27)
+				(color 0 0 255 1)
 			)
 			(justify left bottom)
@@
 			(font
 				(size 1.27 1.27)
+				(color 0 255 0 1)
 			)
 			(justify left bottom)
@@
 				(thickness 0.254)
 				(bold yes)
-				(color 0 132 0 1)
+				(color 0 255 0 1)
 			)
 			(justify left bottom)
@@
 			(font
 				(size 1.27 1.27)
+				(color 255 0 0 1)
 			)
 			(justify left bottom)
@@
 			)
 		)
-		(property "Datasheet" "https://www.ti.com/lit/ds/symlink/lmr54406.pdf?ts=1659688249350&ref_url=https%253A%252F%252Fwww.ti.com%252Fproduct%252FLMR54406%252Fpart-details%252FLMR54406DBVR"
+		(property "Datasheet" "https://www.ti.com/lit/ds/symlink/lmr54406.pdf"
 			(at 161.29 238.1 0)
 			(effects
@@
 		(on_board yes)
 		(dnp no)
-		(fields_autoplaced yes)
 		(property "Reference" "U2"
 			(at 233.68 137.1599 90)
@@
 		)
 		(property "Value" "PEC11L-4220F-S0015"
-			(at 233.68 139.6999 90)
+			(at 220.218 123.698 90)
 			(effects
 				(font
@@
 					(unit 1)
 				)
+			)
+		)
+	)
+	(symbol
+		(lib_id "Mechanical:Fiducial")
+		(at 119.38 193.04 0)
+		(unit 1)
+		(exclude_from_sim no)
+		(in_bom no)
+		(on_board yes)
+		(dnp no)
+		(property "Reference" "FID6"
+			(at 121.92 193.04 0)
+			(effects
+				(font
+					(size 1.27 1.27)
+				)
+				(justify left)
+			)
+		)
+		(property "Value" "Fiducial"
+			(at 121.92 194.31 0)
+			(effects
+				(font
+					(size 1.27 1.27)
+				)
+				(justify left)
+				(hide yes)
+			)
+		)
+		(property "Footprint" "Fiducial:Fiducial_0.75mm_Mask1.5mm"
+			(at 119.38 193.04 0)
+			(effects
+				(font
+					(size 1.27 1.27)
+				)
+				(hide yes)
+			)
+		)
+		(property "Datasheet" "~"
+			(at 119.38 193.04 0)
+			(effects
+				(font
+					(size 1.27 1.27)
+				)
+				(hide yes)
+			)
+		)
+		(property "Description" ""
+			(at 119.38 193.04 0)
+			(effects
+				(font
+					(size 1.27 1.27)
+				)
+				(hide yes)
+			)
+		)
+		(property "Manufacturing comment" "Do Not Place"
+			(at 119.38 193.04 0)
+			(effects
+				(font
+					(size 1.27 1.27)
+				)
+				(hide yes)
+			)
+		)
+		(instances
+			(project "AxxSolder"
+				(path "/d71363c3-4d90-469c-a600-831e2a7cdaef"
+					(reference "FID6")
+					(unit 1)
+				)

Commit message: Cleanup
Parts:
- added D12, D13, D14, D15, D16: LED, LED_SMD:LED_0603_1608Metric, symbol Device:LED
- added R47, R48, R49, R50, R51: 4k7, Resistor_SMD:R_0603_1608Metric, symbol Device:R_Small
Connections:
- net +3.3V: now also D12.2 (A)
- net CURRENT: now also U5.40 (GPIO28_ADC2); no longer U5.39 (GPIO27_ADC1)
- net GND: now also R47.2, R48.2, R49.2, R50.2, R51.2
- net Handle_inp1: now also U5.35 (GPIO23); no longer U5.30 (GPIO19)
- net Handle_inp2: now also U5.36 (GPIO24); no longer U5.31 (GPIO20)
- net Heater: now also U5.38 (GPIO26_ADC0); no longer U5.37 (GPIO25)
- net Stand_inp: now also U5.37 (GPIO25); no longer U5.32 (GPIO21)
- net TC: now also U5.39 (GPIO27_ADC1); no longer U5.38 (GPIO26_ADC0)
- net VBUS: now also D13.2 (A)
- net VBUS_IN: now also U5.41 (GPIO29_ADC3); no longer U5.40 (GPIO28_ADC2)
- net VDD: now also D16.2 (A)
- new net: D12.1 (K), R47.1
- new net: D15.1 (K), R49.1
- new net: D13.1 (K), R48.1
- new net: D14.1 (K), R50.1
- new net: D16.1 (K), R51.1
- new net LED1: D14.2 (A), U5.30 (GPIO19)
- new net LED2: D15.2 (A), U5.31 (GPIO20)

Commit message: Best work yet
Parts:
- removed C10: 10u, Capacitor_SMD:C_0603_1608Metric, symbol Device:C_Small
- removed D4: SMF4L24AT1G, footprints:SODFL3619X98N, symbol SMF4L24AT1G:SMF4L24AT1G
- removed J2: Conn_01x02, Connector_PinHeader_2.54mm:PinHeader_1x02_P2.54mm_Vertical, symbol Connector_Generic:Conn_01x02
- removed J4: 61300611821, Connector_PinHeader_2.54mm:PinHeader_1x06_P2.54mm_Vertical, symbol 61300611821:61300611821
- added D4: LED, LED_SMD:LED_0603_1608Metric, symbol Device:LED
- added J4: Conn_01x07_Pin, Connector_PinHeader_2.54mm:PinHeader_1x07_P2.54mm_Vertical, symbol Connector:Conn_01x07_Pin
- added R52: 4k7, Resistor_SMD:R_0603_1608Metric, symbol Device:R_Small
- added TP1: USR1, TestPoint:TestPoint_Pad_D1.0mm, symbol Connector:TestPoint
- J1: value 284391-7 -> 691243310007; footprint custom_connectors:CONN7_284391-7_TEC -> custom_connectors:691243310007
- U6: value W25Q128JVS -> W25Q16JVSSIQ
Connections:
- net +3.3V: now also U2.1 (S1), J4.7 (Pin_7); no longer U2.2 (S2)
- net BLUE: now also J1.6; no longer J1.5
- net Buzzer: now also U5.36 (GPIO24); no longer U5.4 (GPIO2)
- net CC1: now also IC5.6 (IO4); no longer IC5.1 (IO1)
- net CC2: now also IC5.4 (IO3); no longer IC5.6 (IO4)
- net CURRENT: now also U5.38 (GPIO26_ADC0); no longer U5.40 (GPIO28_ADC2)
- net ENC_A: now also U5.30 (GPIO19); no longer U5.13 (GPIO10)
- net ENC_B: now also U5.29 (GPIO18); no longer U5.8 (GPIO6)
- net GND: now also J1.5, J4.2 (Pin_2), R52.2; no longer J1.6
- net Handle_inp1: now also U5.32 (GPIO21); no longer U5.35 (GPIO23)
- net Handle_inp2: now also U5.34 (GPIO22); no longer U5.36 (GPIO24)
- net Heater: now also U5.37 (GPIO25); no longer U5.38 (GPIO26_ADC0)
- net LED1: now also U5.15 (GPIO12); no longer U5.30 (GPIO19)
- net LED2: now also U5.16 (GPIO13); no longer U5.31 (GPIO20)
- net SCL: now also U5.13 (GPIO10); no longer U5.3 (GPIO1)
- net SDA: now also U5.14 (GPIO11); no longer U5.2 (GPIO0)
- net SPI_CS: now also U5.4 (GPIO2); no longer U5.16 (GPIO13)
- net SPI_DC: now also U5.3 (GPIO1); no longer U5.15 (GPIO12)
- net SPI_MOSI: now also U5.6 (GPIO4); no longer U5.18 (GPIO15)
- net SPI_RST: now also U5.2 (GPIO0); no longer U5.14 (GPIO11)
- net SPI_SCK: now also U5.5 (GPIO3); no longer U5.17 (GPIO14)
- net SW1: now also U2.2 (S2), U5.31 (GPIO20); no longer U2.1 (S1), U5.12 (GPIO9)
- net SW2: now also U5.28 (GPIO17); no longer U5.6 (GPIO4)
- net SW3: now also U5.27 (GPIO16); no longer U5.5 (GPIO3)
- net SWCLK: now also J4.3 (Pin_3)
- net SWDIO: now also J4.4 (Pin_4)
- net Stand_inp: now also U5.35 (GPIO23); no longer U5.37 (GPIO25)
- net USART_RX: now also U5.7 (GPIO5), J4.5 (Pin_5); no longer U5.28 (GPIO17)
- net USART_TX: now also U5.8 (GPIO6), J4.6 (Pin_6); no longer U5.29 (GPIO18)
- net USB_D-: now also IC5.1 (IO1); no longer IC5.4 (IO3)
- net VBUS_IN: now also U5.40 (GPIO28_ADC2); no longer U5.41 (GPIO29_ADC3)
- net ~{USB_BOOT}: now also J4.1 (Pin_1)
- new net: D4.1 (K), R52.1
- new net LED3: D4.2 (A), U5.17 (GPIO14)
- new net USR1: TP1.1, U5.18 (GPIO15)
Other:
- moved on the sheet: D3, IC5

Commit message: Perfection
Parts:
- removed U1: LD1117S33TR_SOT223, Package_TO_SOT_SMD:SOT-223-3_TabPin2, symbol Regulator_Linear:LD1117S33TR_SOT223
- added C10: 100p, Capacitor_SMD:C_0603_1608Metric, symbol Device:C_Small
- added U4: AP2210K-3.3, Package_TO_SOT_SMD:SOT-23-5, symbol Regulator_Linear:AP2204K-3.3
Connections:
- net +3.3V: now also U4.5 (VOUT)
- net +7.5V: now also U4.1 (VIN), U4.3 (EN)
- net GND: now also C10.2, U4.2 (GND)
- new net: C10.1, U4.4 (BYP)
