File: AxxSolder_hardware/AxxSolder.kicad_sch (KiCad schematic)
At the start: 151 parts, among them IC2 OPA2387DSGT, IC3 LMR54406DBVR, IC5 TPD4E1U06DBVR, IC6 STUSB4500QTR, IC8 LTC4440AHMS8E, J1 691243310007, J3 USB4105-GF-A, J4 Conn_01x07_Pin, Q1 STL9P3LLH6, Q3 2N7002NXAKR, U2 PEC11L-4220F-S0015, U3 BSC014N04LS, U4 AP2210K-3.3, U5 RP2040, U6 W25Q16JVSSIQ, Y1 ABM8-272-T3

Commit message: Ordered this one
Parts:
- removed C14, C39, C40, C41, C43, C45, C46, C47, C48, C50: 100n, Capacitor_SMD:C_0603_1608Metric, symbol Device:C
- added C14, C15, C39, C40, C41, C43, C45, C46, C47, C48, C50: 100n, Capacitor_SMD:C_0603_1608Metric, symbol Device:C_Small
- added Q2, Q4, Q5: 2N7002NXAKR, footprints:SOT95P230X110-3N, symbol 2N7002NXAKR:2N7002NXAKR
- added R53: 1M, Resistor_SMD:R_0603_1608Metric, symbol Device:R_Small
- C1, C11, C12, C13, C19, C2, C30, C32, C34, C35, C5, C7, C8: DigiKey PN (none) -> 1276-1869-1-ND; Manufacturer_Name Murata Electronics -> (none); Manufacturer_Part_Number GRM188R6YA106MA73J -> (none); Mouser Part Number 81-GRM188R6YA106MA3J -> (none)
- C10: DigiKey PN (none) -> 1276-1908-1-ND; Manufacturer_Name Murata Electronics -> (none); Manufacturer_Part_Number GRM188R6YA106MA73J -> (none); Mouser Part Number 81-GRM188R6YA106MA3J -> (none)
- C18, C21, C22, C23, C24, C25, C26, C27, C28, C29, C3, C33, C9: DigiKey PN (none) -> 311-1341-1-ND; Manufacturer_Name KEMET -> (none); Manufacturer_Part_Number C0603C104J5RACTU -> (none); Mouser Part Number 80-C0603C104J5R -> (none)
- C36, C38: DigiKey PN (none) -> 311-1060-1-ND
- C37: DigiKey PN (none) -> 399-6708-1-ND; Manufacturer_Name KEMET -> (none); Manufacturer_Part_Number EEV227M035A9MAA -> (none); Mouser Part Number 80-EEV227M035A9MAA -> (none); Mouser Price/Stock https://www.mouser.co.uk/ProductDetail/KEMET/EEV227M035A9MA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 -> (none)
- C4, C6: DigiKey PN (none) -> 399-C0603C102K3RAC7867CT-ND; Manufacturer_Name KEMET -> (none); Manufacturer_Part_Number C0603C102K3GAC -> (none); Mouser Part Number 80-C0603C102K3G -> (none)
- C42, C44: DigiKey PN (none) -> 311-1445-1-ND
- D1: DigiKey PN (none) -> BAV199WQ-7DICT-ND
- D10: DigiKey PN (none) -> 1727-5217-1-ND
- D12, D13, D14, D15, D16, D4: value LED -> 150060VS75000; DigiKey PN (none) -> 732-4980-1-ND
- D2: DigiKey PN (none) -> BAV199WQ-7DICT-ND; Height 1.1 -> (none); Manufacturer_Name Diodes Incorporated -> (none); Manufacturer_Part_Number BAV199WQ-7 -> (none); Mouser Part Number 621-BAV199WQ-7 -> (none); Mouser Price/Stock https://www.mouser.co.uk/ProductDetail/Diodes-Incorporated/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 -> (none)
- D3: DigiKey PN (none) -> 18-SMF4L24AT1GCT-ND; Height 0.98 -> (none); Manufacturer_Name LITTELFUSE -> (none); Manufacturer_Part_Number SMF4L24AT1G -> (none); Mouser Part Number 576-SMF4L24AT1G -> (none)
- D5: value BAT54S -> BAT54SLT1G; DigiKey PN (none) -> BAT54SLT1GOSCT-ND; Manufacturer_Name Diotec Semiconductor -> (none); Manufacturer_Part_Number BAT54S -> (none); Mouser Part Number 637-BAT54S -> (none); Mouser Price/Stock https://www.mouser.co.uk/ProductDetail/Diotec-Semiconductor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 -> (none)
- D6, D7, D8: value BAT54S -> BAT54SLT1G; DigiKey PN (none) -> BAT54SLT1GOSCT-ND
- D9: DigiKey PN (none) -> 1727-5217-1-ND; Height 1.1 -> (none); Manufacturer_Name Nexperia -> (none); Manufacturer_Part_Number PMEG6020ER,115 -> (none); Mouser Part Number 771-PMEG6020ER-115 -> (none); Mouser Price/Stock https://www.mouser.co.uk/ProductDetail/Nexperia/PMEG6020ER1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 -> (none)
- F1: DigiKey PN (none) -> F1229CT-ND; Height 3.81 -> (none); Manufacturer_Name LITTELFUSE -> (none); Manufacturer_Part_Number 0154007.DR -> (none); Mouser Part Number 576-0154007.DR -> (none)
- FB1: DigiKey PN (none) -> 490-5214-1-ND; Height 0.95 -> (none); Manufacturer_Name Murata Electronics -> (none); Manufacturer_Part_Number BLM18HE601SN1D -> (none); Mouser Part Number 81-BLM18HE601SN1D -> (none); Mouser Price/Stock https://www.mouser.co.uk/ProductDetail/Murata-Electronics/B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 -> (none)
- IC2: DigiKey PN (none) -> 296-OPA2387DSGTCT-ND; Height 0.8 -> (none); Manufacturer_Name Texas Instruments -> (none); Manufacturer_Part_Number OPA2387DSGT -> (none); Mouser Part Number 595-OPA2387DSGT -> (none); Mouser Price/Stock https://www.mouser.co.uk/ProductDetail/Texas-Instruments/OP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 -> (none)
- IC3: DigiKey PN (none) -> 296-LMR54406DBVRCT-ND; Height 1.45 -> (none); Manufacturer_Name Texas Instruments -> (none); Manufacturer_Part_Number LMR54406DBVR -> (none); Mouser Part Number 595-LMR54406DBVR -> (none); Mouser Price/Stock https://www.mouser.co.uk/ProductDetail/Texas-Instruments/LM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 -> (none)
- IC5: DigiKey PN (none) -> TPD4E1U06DBVR; Height 1.45 -> (none); Manufacturer_Name Texas Instruments -> (none); Manufacturer_Part_Number TPD4E1U06DBVR -> (none); Mouser Part Number 595-TPD4E1U06DBVR -> (none); Mouser Price/Stock https://www.mouser.co.uk/ProductDetail/Texas-Instruments/TP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 -> (none)
- IC6: DigiKey PN (none) -> 497-18060-1-ND; Height 1 -> (none); Manufacturer_Name STMicroelectronics -> (none); Manufacturer_Part_Number STUSB4500QTR -> (none); Mouser Part Number 511-STUSB4500QTR -> (none); Mouser Price/Stock https://www.mouser.co.uk/ProductDetail/STMicroelectronics/S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 -> (none)
- IC8: DigiKey PN (none) -> 505-LTC4440AHMS8E-5#PBF-ND; Height 1.1 -> (none); Manufacturer_Name Analog Devices -> (none); Manufacturer_Part_Number LTC4440AHMS8E-5#PBF -> (none); Mouser Part Number 584-C4440AHMS8E-5PBF -> (none); Mouser Price/Stock https://www.mouser.co.uk/ProductDetail/Analog-Devices/LTC44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 -> (none)
- J1: DigiKey PN (none) -> 732-691243310007-ND
- J3: DigiKey PN (none) -> 2073-USB4105-GF-ACT-ND; MANUFACTURER Global Connector Technology -> (none); MAXIMUM_PACKAGE_HEIGHT 3.31mm -> (none); PARTREV B3 -> (none); STANDARD Manufacturer Recommendations -> (none)
- L1: DigiKey PN (none) -> 118-SRP7028CC-150MCT-ND; Height 3 -> (none); Manufacturer_Name Bourns -> (none); Manufacturer_Part_Number SRP7028CC-150M -> (none); Mouser Part Number 652-SRP7028CC-150M -> (none); Mouser Price/Stock https://www.mouser.co.uk/ProductDetail/Bourns/SRP7028CC-150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 -> (none)
- LS1: DigiKey PN (none) -> 102-3737-1-ND; Height 5 -> (none); Manufacturer_Name CUI Devices -> (none); Manufacturer_Part_Number CMI-9653S-SMT-TR -> (none); Mouser Part Number 490-CMI-9653S-SMT-TR -> (none); Mouser Price/Stock https://www.mouser.co.uk/ProductDetail/CUI-Devices/CMI-9653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 -> (none)
- Q1: DigiKey PN (none) -> 497-17897-1-ND; Manufacturer_Name STMicroelectronics -> (none); Manufacturer_Part_Number STL9P3LLH6 -> (none); Mouser Part Number 511-STL9P3LLH6 -> (none); Mouser Price/Stock https://www.mouser.co.uk/ProductDetail/STMicroelectronics/S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 -> (none)
- Q3: DigiKey PN (none) -> 2N7002NXAKR
- R1, R14, R17, R5: DigiKey PN (none) -> 311-1.50KHRCT-ND
- R10, R3: DigiKey PN (none) -> 311-220KHRCT-ND
- R11, R12, R15, R21, R24: DigiKey PN (none) -> 311-22.0KHRCT-ND
- R13, R34: DigiKey PN (none) -> P100HCT-ND
- R16, R43: DigiKey PN (none) -> 311-1.00KHRCT-ND
- R18, R19, R20, R22, R23, R25, R26, R27, R28, R29, R30, R31, R32, R33, R35, R36, R37, R38, R4, R6: DigiKey PN (none) -> 311-4.70KHRCT-ND
- R2, R7, R8, R9: DigiKey PN (none) -> 311-360KHRCT-ND
- R42: DigiKey PN (none) -> 541-10153-1-ND; Height 0.889 -> (none); Manufacturer_Name Vishay -> (none); Manufacturer_Part_Number WSLP25125L000FEA -> (none); Mouser Part Number 71-WSLP25125L000FEA -> (none); Mouser Price/Stock https://www.mouser.co.uk/ProductDetail/Vishay-Dale/WSLP2512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 -> (none)
- R44: DigiKey PN (none) -> 311-10.0KHRCT-ND
- R45, R46: DigiKey PN (none) -> CR0603-FX-27R0ELFCT-ND
- R47, R49, R50, R52: value 4k7 -> 100; DigiKey PN (none) -> P100HCT-ND
- R48, R51: value 4k7 -> 1k5; footprint Resistor_SMD:R_0603_1608Metric -> Resistor_SMD:R_0603_1608Metric_Pad0.98x0.95mm_HandSolder; DigiKey PN (none) -> 311-1.50KHRCT-ND
- S2, S3: DigiKey PN (none) -> 679-ADTSM644RVTRCT-ND; Height 7.3 -> (none); Manufacturer_Name Apem -> (none); Manufacturer_Part_Number ADTSM644RVTR -> (none); Mouser Part Number 642-ADTSM644RVTR -> (none)
- U2: DigiKey PN (none) -> PEC11L-4220F-S0015-ND; Height 25 -> (none); Manufacturer_Name Bourns -> (none); Manufacturer_Part_Number PEC11L-4220F-S0015 -> (none); Mouser Part Number 652-PEC11L4220FS0015 -> (none); Mouser Price/Stock https://www.mouser.co.uk/ProductDetail/Bourns/PEC11L-4220F-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 -> (none)
- U3: DigiKey PN (none) -> BSC014N04LSATMA1CT-ND; Manufacturer_Name Infineon Technologies -> (none); Manufacturer_Part_Number BSC014N04LSATMA1 -> (none); Mouser Part Number 726-BSC014N04LSATMA1 -> (none)
- U4: value AP2210K-3.3 -> AP2210K-3.3TRG1; DigiKey PN (none) -> AP2210K-3.3TRG1DICT-ND
- U5: DigiKey PN (none) -> 2648-SC0914(13)CT-ND
- U6: DigiKey PN (none) -> W25Q16JVSSIQ-ND
- Y1: DigiKey PN (none) -> 535-ABM8-272-T3CT-ND
Connections:
- net +1V1: now also C40.1, C41.1
- net +3.3V: now also D14.2 (A), D15.2 (A), D4.2 (A), C14.1, C39.1, C43.1, C45.1, C46.1, C47.1, C48.1, C50.1
- net +7.5V: now also C7.1, C8.1; no longer C7.2, C8.2
- net BLUE: now also J1.5; no longer J1.6
- net BOOST: now also C30.1; no longer C30.2
- net GND: now also C11.1, C12.1, C13.1, C34.2, C35.2, C5.2, C7.2, C8.2, J1.6, C14.2, C15.1, C39.2, C40.2, C41.2, C43.2, C45.2, C46.2, C47.2, C48.2, C50.2, Q2.2 (S), Q4.2 (S), Q5.2 (S), R53.2; no longer C11.2, C12.2, C13.2, C34.1, C35.1, C5.1, C7.1, C8.1, J1.5, J3.SH1 (SHELL_GND), J3.SH2 (SHELL_GND__1), J3.SH3 (SHELL_GND__2), J3.SH4 (SHELL_GND__3), R49.2, R50.2, R52.2
- net LED1: now also Q5.1 (G); no longer D14.2 (A)
- net LED2: now also Q4.1 (G); no longer D15.2 (A)
- net LED3: now also Q2.1 (G); no longer D4.2 (A)
- net RED: now also C30.2; no longer C30.1
- net VBUS: now also C11.2; no longer C11.1
- net VDD: now also C34.1, C35.1, C5.1; no longer C34.2, C35.2, C5.2
- net VDD_IN: now also C9.1; no longer C9.2
- net at R13.2: now also C9.2; no longer C9.1
- net at IC6.21 (VREG_1V2): now also C13.2; no longer C13.1
- net at IC6.23 (VREG_2V7): now also C12.2; no longer C12.1
- new net: Q5.3 (D), R49.2
- new net: Q4.3 (D), R50.2
- new net: Q2.3 (D), R52.2
- new net: C15.2, J3.SH1 (SHELL_GND), J3.SH2 (SHELL_GND__1), J3.SH3 (SHELL_GND__2), J3.SH4 (SHELL_GND__3), R53.1
Other:
- moved on the sheet: D12, D13, D14, D15, D16, D4, R1, R14, R47, R48, R49, R5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
